Commit message: updates

File: openarm_bimanual_description/urdf/openarm_bimanual.urdf (robot description, URDF)
Before this commit: robot openarm_bimanual, 40 links, 39 joints
Links:
- link right_link1: geometry collision box size=0.11 0.073 0.0592; visual mesh filename=package://openarm_description/meshes/right_base_link_color.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

File: openarm_bimanual_description/urdf/openarm_bimanual_cameraMount.xacro (robot description, xacro)
@@ -13,5 +13,5 @@
 -->
 <robot xmlns:xacro="http://www.ros.org/wiki/xacro">
-    <xacro:include filename="$(find camAssembly_4H_description)/urdf/cameraMount.urdf.xacro"/>
+    <xacro:include filename="$(find camAssembly_4H_description)/urdf/camAssembly_4H.urdf.xacro"/>
     <xacro:cam_mount parent="pedestal_link"/>
 </robot>

File: openarm_description/urdf/openarm.urdf (robot description, URDF)
Before this commit: robot openarm, 12 links, 11 joints
Links:
- link link1: geometry collision box size=0.11 0.073 0.0592; visual mesh filename=package://openarm_description/meshes/right_base_link_color.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

File: openarm_description/urdf/openarm.urdf.xacro (robot description, xacro)
@@ -18,4 +18,4 @@
     <xacro:include filename="openarm.xacro"/>
     <xacro:openarm prefix="$(arg prefix)" use_mock_hardware="$(arg use_mock_hardware)" mock_sensor_commands="$(arg mock_sensor_commands)"/>
-    <xacro:include filename="$(find openarm_description)/urdf/openarm_sensors.xacro"/>
+    <!-- <xacro:include filename="$(find openarm_description)/urdf/openarm_sensors.xacro"/> -->
 </robot>

File: openarm_description/urdf/openarm.xacro (robot description, xacro)
@@ -35,9 +35,9 @@
         <link name="${prefix}link1">
             <visual>
-                <origin rpy="0 0 0" xyz="0.0 0.0 -0.0007"/>
-                <geometry>
-                    <mesh filename="package://openarm_description/meshes/link1.stl"/>
-                </geometry>
-                <material name="gray"/>
+                <origin rpy="0 0 0" xyz="0.0 0.0 0.07"/>
+                <geometry>
+                <mesh filename="package://openarm_description/meshes/right_base.dae" scale= "0.001 0.001 0.001"/>
+                </geometry>
+                <!-- <material name="gray"/> -->
             </visual>
             <collision>
