Commit message: Updated URDF and moveit setup

File: openarm_description/urdf/arm/openarm_arm.xacro (robot description, xacro)
@@ -37,4 +37,5 @@
     </joint>
     <xacro:link_with_sc no_prefix="${no_prefix}" name="link2" gazebo="${gazebo}" kinematics_link="${kinematics_link}" reflect="${reflect}"/>
+    <xacro:property name="limit_offset_joint2" value="0.0" />
     <xacro:if value="${prefix.find('right_') != -1}">
       <xacro:property name="limit_offset_joint2" value="${pi/2}" />

File: openarm_description/urdf/robot/v10.urdf.xacro (robot description, xacro)
@@ -23,9 +23,9 @@
   <xacro:arg name="rpy" default="0 0 0" />
   <!-- Is the robot being controlled with ros2_control?" -->
-  <xacro:arg name="ros2_control" default="false" />
+  <xacro:arg name="ros2_control" default="true" />
   <!-- IP address or hostname of the robot" -->
   <xacro:arg name="can" default="can0" />
   <!-- Should a fake hardware be used? -->
-  <xacro:arg name="use_fake_hardware" default="false" />
+  <xacro:arg name="use_fake_hardware" default="true" />
   <!-- Should fake sensors be used? -->
   <xacro:arg name="fake_sensor_commands" default="false" />
