Commit message: new URDF

File: openarm_description/urdf/robot/openarm_robot.xacro (robot description, xacro)
@@ -77,4 +77,5 @@
         kinematics_link="${kinematics_link}"
         kinematics_offset="${kinematics_offset}" />
+        <xacro:if value="${ros2_control}">
         <xacro:openarm_arm_ros2_control
         arm_type="${arm_type}"
@@ -87,5 +88,6 @@
         hand="${hand}"
         bimanual="true"
-      />
+        />
+       </xacro:if>
         <!-- right arm -->
         <xacro:openarm_arm
@@ -103,18 +105,19 @@
         kinematics_link="${kinematics_link}"
         kinematics_offset="${kinematics_offset}" />
-        <xacro:openarm_arm_ros2_control
-        arm_type="${arm_type}"
-        arm_prefix="right_"
-        can="can0"
-        use_fake_hardware="${use_fake_hardware}"
-        fake_sensor_commands="${fake_sensor_commands}"
-        gazebo="${gazebo}"
-        gazebo_effort="${gazebo_effort}"
-        hand="${hand}"
-        bimanual="true"
-        />
+        <xacro:if value="${ros2_control}">
+            <xacro:openarm_arm_ros2_control
+            arm_type="${arm_type}"
+            arm_prefix="right_"
+            can="can0"
+            use_fake_hardware="${use_fake_hardware}"
+            fake_sensor_commands="${fake_sensor_commands}"
+            gazebo="${gazebo}"
+            gazebo_effort="${gazebo_effort}"
+            hand="${hand}"
+            bimanual="true"/>
+        </xacro:if>
         <xacro:if value="${hand and ee_type == 'openarm_hand'}">
             <xacro:openarm_hand
-                connected_to="left_${arm_type}_link8"
+                connected_to="openarm_left_link8"
                 arm_type="${arm_type}"
                 arm_prefix="left_"
@@ -130,5 +133,5 @@
             />
             <xacro:openarm_hand
-                connected_to="right_${arm_type}_link8"
+                connected_to="openarm_right_link8"
                 arm_type="${arm_type}"
                 arm_prefix="right_"
@@ -159,4 +162,5 @@
         connected_to=""
         />
+        <xacro:if value="${ros2_control}">
         <xacro:openarm_arm_ros2_control
             arm_type="${arm_type}"
@@ -168,9 +172,10 @@
             gazebo_effort="${gazebo_effort}"
             hand="${hand}"
-            bimanual="false"
-        />
+            bimanual="false"/>
+        </xacro:if>
         <xacro:if value="${hand and ee_type == 'openarm_hand'}">
         <xacro:property name="special_connection" value="$(arg special_connection)" />
-        <xacro:property name="connection" value="${special_connection if special_connection != '' else arm_type + '_link8'}" />
+        <!-- <xacro:property name="connection" value="${special_connection if special_connection != '' else arm_type + '_link8'}" /> -->
+        <xacro:property name="connection" value="${special_connection if special_connection != '' else 'openarm' + '_link8'}" />
         <xacro:openarm_hand
             connected_to="${arm_prefix_modified}${connection}"
@@ -185,6 +190,5 @@
             tcp_rpy="$(arg tcp_rpy)"
             gazebo="${gazebo}"
-            description_pkg="$(arg description_pkg)"
-        />
+            description_pkg="$(arg description_pkg)"/>
         </xacro:if>
         <!-- <xacro:if value="${hand and ee_type != 'none' and ee_type != 'openarm_hand'}">
